Commit message: 发现错误在于collision坐标与方向不正确

File: raisimOgre/examples/rsc/dancer_model/dancer_urdf_model.urdf (robot description, URDF)
Before this commit: robot dancer_urdf_model, 22 links, 21 joints
Links:
- link arm_left: geometry collision box size=0.06 0.16 0.06; visual mesh filename=arm_left.stl
- link arm_right: geometry collision box size=0.06 0.16 0.06; visual mesh filename=arm_right.stl
- link body_chest: geometry collision box size=0.1 0.14 0.08; visual mesh filename=body_chest.stl
